Commit message: make available the spawn of the full_fake_grippers and no_grippers

File: talos_description/robots/talos_arm_right.urdf.xacro (robot description, xacro)
@@ -21,4 +21,5 @@
   <xacro:include filename="$(find talos_description)/urdf/sensors/ftsensor.urdf.xacro" />
   <xacro:include filename="$(find talos_description)/urdf/gripper/gripper.urdf.xacro" />
+  <xacro:include filename="$(find talos_description_calibration)/urdf/calibration/calibration_constants.urdf.xacro" />
   <xacro:arg name="use_sim" default="false"/>
   <xacro:arg name="robot_model" default="arm_right"/>

File: talos_description/ros2_control/ros2_control.urdf.xacro (robot description, xacro)
@@ -17,8 +17,14 @@
     <xacro:arg name="robot_model" default="$(arg robot_model)"/> <!-- full_fake_grippers,
                                         full_no_grippers, full_v1, full_v2, lower_body_torso_head, lower_body -->
-  <xacro:include filename="$(find talos_description)/urdf/sensors/ftsensor.ros2_control.xacro" />
+    <xacro:include filename="$(find talos_description)/urdf/sensors/ftsensor.ros2_control.xacro" />
     <xacro:include filename="$(find talos_description)/urdf/arm/arm.ros2_control.xacro" />
     <xacro:include filename="$(find talos_description)/urdf/arm/wrist.ros2_control.xacro"/>
     <xacro:include filename="$(find talos_description)/urdf/gripper/gripper.ros2_control.xacro" />
+    <xacro:include filename="$(find talos_description)/urdf/head/head.ros2_control.xacro" />
+    <xacro:include filename="$(find talos_description)/urdf/leg/leg.ros2_control.xacro" />
+    <!-- Calibration offsets -->
+    <xacro:include filename="$(find talos_description_calibration)/urdf/calibration/calibration_constants.urdf.xacro" />
+    <xacro:property name="leg_reduction"    value="1.0" />
+    <xacro:property name="flexibility"    value="false" />
     <ros2_control name="ros2_control_talos_system" type="system">
       <hardware>
@@ -30,23 +36,51 @@
         </xacro:unless>
       </hardware>
-      <!-- IMU
+      <!-- IMU -->
       <xacro:if value="$(arg use_sim)">
         <xacro:ros2_control_imu name="base_imu_sensor"/>
-      </xacro:if>-->
-    <xacro:if value="${robot_model == 'arm_right'}">
+      </xacro:if>
       <!-- arm right-->
-      <xacro:ros2_control_arm name="arm" side="right" number="1"/>
-      <xacro:ros2_control_arm name="arm" side="right" number="2"/>
-      <xacro:ros2_control_arm name="arm" side="right" number="3"/>
-      <xacro:ros2_control_arm name="arm" side="right" number="4"/>
-     </xacro:if>
-    <!-- Wrist -->
-    <xacro:ros2_control_wrist name="arm" side="right" number="5"/>
-    <xacro:ros2_control_wrist name="arm" side="right" number="6"/>
-    <xacro:ros2_control_wrist name="arm" side="right" number="7"/>
-    <!-- Gripper right-->
-    <xacro:ros2_control_gripper name="gripper_right"/>
-     <!-- Force Torque sensor-->
-    <xacro:ros2_control_force_torque_sensor name="wrist_right_ft_sensor"/>
+      <xacro:if value="${robot_model in ['arm_right', 'full_fake_grippers']}">
+        <xacro:ros2_control_arm name="arm" side="right" number="1"/>
+        <xacro:ros2_control_arm name="arm" side="right" number="2"/>
+        <xacro:ros2_control_arm name="arm" side="right" number="3"/>
+        <xacro:ros2_control_arm name="arm" side="right" number="4"/>
+      </xacro:if>
+      <!-- Wrist right -->
+      <xacro:ros2_control_wrist name="arm" side="right" number="5"/>
+      <xacro:ros2_control_wrist name="arm" side="right" number="6"/>
+      <xacro:ros2_control_wrist name="arm" side="right" number="7"/>
+      <!-- Arm left-->
+      <xacro:ros2_control_arm name="arm" side="left" number="1"/>
+      <xacro:ros2_control_arm name="arm" side="left" number="2"/>
+      <xacro:ros2_control_arm name="arm" side="left" number="3"/>
+      <xacro:ros2_control_arm name="arm" side="left" number="4"/>
+      <!-- Wrist left -->
+      <xacro:ros2_control_wrist name="arm" side="left" number="5"/>
+      <xacro:ros2_control_wrist name="arm" side="left" number="6"/>
+      <xacro:ros2_control_wrist name="arm" side="left" number="7"/>
+      <!-- Gripper right-->
+      <xacro:ros2_control_gripper name="gripper_right"/>
+      <!-- Gripper left-->
+      <xacro:ros2_control_gripper name="gripper_left"/>
+      <!-- Head -->
+      <xacro:ros2_control_head name="head" offset_value_1="${head_1_joint_yaw_offset}" offset_value_2="${head_2_joint_yaw_offset}"/>
+       <!-- Force Torque sensor-->
+      <xacro:ros2_control_force_torque_sensor name="wrist_right_ft_sensor"/>
+      <xacro:ros2_control_force_torque_sensor name="wrist_left_ft_sensor"/>
+      <!-- Leg left -->
+      <xacro:ros2_control_leg side="left" number="1" leg_reduction="${leg_reduction}" />
+      <xacro:ros2_control_leg side="left" number="2" leg_reduction="${leg_reduction}" />
+      <xacro:ros2_control_leg side="left" number="3" leg_reduction="${leg_reduction}" />
+      <xacro:ros2_control_leg side="left" number="4" leg_reduction="${leg_reduction}" />
+      <xacro:ros2_control_leg side="left" number="5" leg_reduction="${leg_reduction}" />
+      <xacro:ros2_control_leg side="left" number="6" leg_reduction="${leg_reduction}" />
+      <!-- Leg right -->
+      <xacro:ros2_control_leg side="right" number="1" leg_reduction="${leg_reduction}" />
+      <xacro:ros2_control_leg side="right" number="2" leg_reduction="${leg_reduction}" />
+      <xacro:ros2_control_leg side="right" number="3" leg_reduction="${leg_reduction}" />
+      <xacro:ros2_control_leg side="right" number="4" leg_reduction="${leg_reduction}" />
+      <xacro:ros2_control_leg side="right" number="5" leg_reduction="${leg_reduction}" />
+      <xacro:ros2_control_leg side="right" number="6" leg_reduction="${leg_reduction}" />
     </ros2_control>
   </xacro:macro>

Commit message: visualization complete for all the models of TALOS

File: talos_description/robots/talos_arm_right.urdf.xacro (robot description, xacro)
@@ -23,5 +23,4 @@
   <xacro:include filename="$(find talos_description_calibration)/urdf/calibration/calibration_constants.urdf.xacro" />
   <xacro:arg name="use_sim" default="false"/>
-  <xacro:arg name="robot_model" default="arm_right"/>
   <xacro:arg name="multiple" default="false"/>
   <xacro:property name="is_multiple" value="$(arg multiple)" />
@@ -59,10 +58,10 @@
   <xacro:ft_sensor name="wrist" parent="arm_right_7_link" side="right" reflect="1"  />
   <xacro:talos_gripper name="gripper_right" parent="wrist_right_ft_tool_link" reflect="-1" />
-  <!-- ROS 2 Control-->
-  <xacro:include filename="$(find talos_description)/ros2_control/ros2_control.urdf.xacro" />
-  <xacro:talos_ros2_control use_sim="$(arg use_sim)" robot_model="$(arg robot_model)"/>
   <!-- Generic simulator_gazebo plugins -->
   <xacro:include filename="$(find talos_description)/gazebo/gazebo.urdf.xacro" />
   <!-- Materials for visualization -->
   <xacro:include filename="$(find talos_description)/urdf/materials.urdf.xacro" />
+  <!-- ROS 2 Control-->
+  <xacro:include filename="$(find talos_description)/ros2_control/ros2_control.urdf.xacro" />
+  <xacro:talos_ros2_control use_sim="$(arg use_sim)"/>
 </robot>

File: talos_description/robots/talos_full_fake_grippers.urdf.xacro (robot description, xacro)
@@ -81,4 +81,4 @@
 <!-- ROS 2 Control-->
 <xacro:include filename="$(find talos_description)/ros2_control/ros2_control.urdf.xacro" />
-<xacro:talos_ros2_control use_sim="$(arg use_sim)" robot_model="full_fake_grippers"/>
+<xacro:talos_ros2_control use_sim="$(arg use_sim)"/>
 </robot>

File: talos_description/robots/talos_lower_body.urdf.xacro (robot description, xacro)
@@ -11,11 +11,4 @@
         xmlns:controller="http://playerstage.sourceforge.net/gazebo/xmlschema/#controller"
         xmlns:interface="http://playerstage.sourceforge.net/gazebo/xmlschema/#interface">
-  <xacro:if value="$(arg enable_crane)">
-    <xacro:include filename="$(find talos_description)/urdf/crane/crane.urdf.xacro" />
-  </xacro:if>
-  <xacro:include filename="$(find talos_description)/urdf/torso/torso.urdf.xacro" />
-  <xacro:include filename="$(find talos_description)/urdf/head/head.urdf.xacro" />
-  <xacro:include filename="$(find talos_description)/urdf/arm/arm_specifics_v2.urdf.xacro" />
-  <xacro:include filename="$(find talos_description)/urdf/arm/arm.urdf.xacro" />
   <xacro:include filename="$(find talos_description)/urdf/sensors/ftsensor.urdf.xacro" />
   <xacro:include filename="$(find talos_description)/urdf/leg/leg.urdf.xacro" />
@@ -23,16 +16,32 @@
   <xacro:include filename="$(find talos_description_inertial)/urdf/inertial.xacro" />
   <xacro:include filename="$(find talos_description)/urdf/extras/addons.urdf.xacro" />
-  <xacro:talos_torso name="torso" />
   <xacro:arg name="use_sim" default="false"/>
   <xacro:arg name="multiple" default="false"/>
   <xacro:property name="is_multiple" value="$(arg multiple)" />
-  <xacro:if value="$(arg enable_crane)">
-    <xacro:crane parent="torso_2_link"/>
-  </xacro:if>
-  <xacro:talos_head name="head" parent="torso_2_link" disable_gazebo_camera="$(arg disable_gazebo_camera)"/>
-  <xacro:talos_arm name="arm" parent="torso_2_link" side="left" reflect="1"/>
-  <xacro:talos_arm name="arm" parent="torso_2_link" side="right" reflect="-1"/>
-  <xacro:ft_sensor name="wrist" parent="arm_right_7_link" side="right" reflect="1"  />
-  <xacro:ft_sensor name="wrist" parent="arm_left_7_link"  side="left"  reflect="-1" />
+  <!--************************-->
+  <!--        BASE_LINK       -->
+  <!--************************-->
+  <link name="base_link">
+    <inertial>
+      <origin xyz="-0.08222 0.00838 -0.07261" rpy="0.00000 0.00000 0.00000"/>
+      <mass value="13.53810"/>
+      <inertia ixx="0.06989000000" ixy="-0.00011700000" ixz="0.00023000000"
+               iyy="0.03998200000" iyz="-0.00132500000"
+               izz="0.08234500000"/>
+    </inertial>
+   <visual>
+      <origin xyz="0 0 0" rpy="0 0 0" />
+      <geometry>
+        <mesh filename="package://talos_description/meshes/torso/base_link.STL" scale="1 1 1"/>
+      </geometry>
+      <material name="LightGrey" />
+    </visual>
+   <collision>
+      <origin xyz="0 0 0" rpy="0 0 0" />
+      <geometry>
+        <mesh filename="package://talos_description/meshes/torso/base_link_collision.STL" scale="1 1 1"/>
+      </geometry>
+    </collision>
+  </link>
   <xacro:talos_leg prefix="left"  reflect="1" />
   <xacro:talos_leg prefix="right" reflect="-1" />

File: talos_description/robots/talos_lower_body_torso_head.urdf.xacro (robot description, xacro)
@@ -14,27 +14,24 @@
     <xacro:include filename="$(find talos_description)/urdf/crane/crane.urdf.xacro" />
   </xacro:if>
-  <xacro:include filename="$(find talos_description)/urdf/torso/torso.urdf.xacro" />
-  <xacro:include filename="$(find talos_description)/urdf/head/head.urdf.xacro" />
-  <xacro:include filename="$(find talos_description)/urdf/arm/arm_specifics_v2.urdf.xacro" />
-  <xacro:include filename="$(find talos_description)/urdf/arm/arm.urdf.xacro" />
   <xacro:include filename="$(find talos_description)/urdf/sensors/ftsensor.urdf.xacro" />
   <xacro:include filename="$(find talos_description)/urdf/leg/leg.urdf.xacro" />
   <xacro:include filename="$(find talos_description)/urdf/leg/foot_collision_$(arg foot_collision).urdf.xacro" />
   <xacro:include filename="$(find talos_description_inertial)/urdf/inertial.xacro" />
+  <xacro:include filename="$(find talos_description)/urdf/torso/torso.urdf.xacro" />
+  <xacro:include filename="$(find talos_description)/urdf/head/head.urdf.xacro" />
   <xacro:include filename="$(find talos_description)/urdf/extras/addons.urdf.xacro" />
+  <!--************************-->
+  <!--        BASE_LINK       -->
+  <!--************************-->
   <xacro:talos_torso name="torso" />
+  <xacro:talos_head name="head" parent="torso_2_link" disable_gazebo_camera="$(arg disable_gazebo_camera)"/>
   <xacro:arg name="use_sim" default="false"/>
   <xacro:arg name="multiple" default="false"/>
   <xacro:property name="is_multiple" value="$(arg multiple)" />
+  <xacro:talos_leg prefix="left"  reflect="1" />
+  <xacro:talos_leg prefix="right" reflect="-1" />
   <xacro:if value="$(arg enable_crane)">
     <xacro:crane parent="torso_2_link"/>
   </xacro:if>
-  <xacro:talos_head name="head" parent="torso_2_link" disable_gazebo_camera="$(arg disable_gazebo_camera)"/>
-  <xacro:talos_arm name="arm" parent="torso_2_link" side="left" reflect="1"/>
-  <xacro:talos_arm name="arm" parent="torso_2_link" side="right" reflect="-1"/>
-  <xacro:ft_sensor name="wrist" parent="arm_right_7_link" side="right" reflect="1"  />
-  <xacro:ft_sensor name="wrist" parent="arm_left_7_link"  side="left"  reflect="-1" />
-  <xacro:talos_leg prefix="left"  reflect="1" />
-  <xacro:talos_leg prefix="right" reflect="-1" />
   <!-- Macro to have the add-on links specific to each TALOS -->
   <xacro:talos_addons />

File: talos_description/ros2_control/ros2_control.urdf.xacro (robot description, xacro)
@@ -14,7 +14,5 @@
 <robot xmlns:xacro="http://ros.org/wiki/xacro"
        name="talos" >
-  <xacro:macro name="talos_ros2_control" params="use_sim:=^|false robot_model:=arm_right">
-    <xacro:arg name="robot_model" default="$(arg robot_model)"/> <!-- full_fake_grippers,
-                                        full_no_grippers, full_v1, full_v2, lower_body_torso_head, lower_body -->
+  <xacro:macro name="talos_ros2_control" params="use_sim:=^|false">
     <xacro:include filename="$(find talos_description)/urdf/sensors/ftsensor.ros2_control.xacro" />
     <xacro:include filename="$(find talos_description)/urdf/arm/arm.ros2_control.xacro" />
@@ -25,6 +23,5 @@
     <!-- Calibration offsets -->
     <xacro:include filename="$(find talos_description_calibration)/urdf/calibration/calibration_constants.urdf.xacro" />
-    <xacro:property name="leg_reduction"    value="1.0" />
-    <xacro:property name="flexibility"    value="false" />
+    <xacro:property name="leg_reduction"    value="1.0" /><!-- i don't like here-->
     <ros2_control name="ros2_control_talos_system" type="system">
       <hardware>
@@ -41,10 +38,8 @@
       </xacro:if>
       <!-- arm right-->
-      <xacro:if value="${robot_model in ['arm_right', 'full_fake_grippers']}">
-        <xacro:ros2_control_arm name="arm" side="right" number="1"/>
-        <xacro:ros2_control_arm name="arm" side="right" number="2"/>
-        <xacro:ros2_control_arm name="arm" side="right" number="3"/>
-        <xacro:ros2_control_arm name="arm" side="right" number="4"/>
-      </xacro:if>
+      <xacro:ros2_control_arm name="arm" side="right" number="1"/>
+      <xacro:ros2_control_arm name="arm" side="right" number="2"/>
+      <xacro:ros2_control_arm name="arm" side="right" number="3"/>
+      <xacro:ros2_control_arm name="arm" side="right" number="4"/>
       <!-- Wrist right -->
       <xacro:ros2_control_wrist name="arm" side="right" number="5"/>

File: talos_description/urdf/talos_full_common.urdf.xacro (robot description, xacro)
@@ -16,7 +16,7 @@
   <xacro:include filename="$(find talos_description)/urdf/torso/torso.urdf.xacro" />
   <xacro:include filename="$(find talos_description)/urdf/head/head.urdf.xacro" />
-  <xacro:include filename="$(find talos_description)/urdf/arm/arm_specifics_v2.urdf.xacro" />
   <xacro:include filename="$(find talos_description)/urdf/arm/arm.urdf.xacro" />
   <xacro:include filename="$(find talos_description)/urdf/sensors/ftsensor.urdf.xacro" />
+  <xacro:include filename="$(find talos_description)/urdf/gripper/gripper.urdf.xacro" />
   <xacro:include filename="$(find talos_description)/urdf/leg/leg.urdf.xacro" />
   <xacro:include filename="$(find talos_description)/urdf/leg/foot_collision_$(arg foot_collision).urdf.xacro" />
@@ -24,17 +24,19 @@
   <xacro:include filename="$(find talos_description)/urdf/extras/addons.urdf.xacro" />
   <xacro:talos_torso name="torso" />
+  <xacro:if value="$(arg enable_crane)">
+    <xacro:crane parent="torso_2_link"/>
+  </xacro:if>
   <xacro:arg name="use_sim" default="false"/>
   <xacro:arg name="multiple" default="false"/>
   <xacro:property name="is_multiple" value="$(arg multiple)" />
-  <xacro:if value="$(arg enable_crane)">
-    <xacro:crane parent="torso_2_link"/>
-  </xacro:if>
-  <xacro:talos_head name="head" parent="torso_2_link" disable_gazebo_camera="$(arg disable_gazebo_camera)"/>
-  <xacro:talos_arm name="arm" parent="torso_2_link" side="left" reflect="1"/>
-  <xacro:talos_arm name="arm" parent="torso_2_link" side="right" reflect="-1"/>
+  <xacro:talos_head name="head" parent="torso_2_link" disable_gazebo_camera="$(arg disable_gazebo_camera)" head_type="$(arg head_type)"/>
+  <xacro:talos_arm name="arm" parent="torso_2_link" side="left" reflect="1" />
+  <xacro:talos_arm name="arm" parent="torso_2_link" side="right" reflect="-1" />
   <xacro:ft_sensor name="wrist" parent="arm_right_7_link" side="right" reflect="1"  />
   <xacro:ft_sensor name="wrist" parent="arm_left_7_link"  side="left"  reflect="-1" />
-  <xacro:talos_leg prefix="left"  reflect="1" />
-  <xacro:talos_leg prefix="right" reflect="-1" />
+  <xacro:talos_gripper name="gripper_left" parent="wrist_left_ft_tool_link" reflect="1" />
+  <xacro:talos_gripper name="gripper_right" parent="wrist_right_ft_tool_link" reflect="-1" />
+  <xacro:talos_leg prefix="left"  reflect="1" flexibility="$(arg flexibility)"/>
+  <xacro:talos_leg prefix="right" reflect="-1" flexibility="$(arg flexibility)"/>
   <!-- Macro to have the add-on links specific to each TALOS -->
   <xacro:talos_addons />
