Commit message: working version with default position controllers

File: talos_description/robots/talos_lower_body.urdf.xacro (robot description, xacro)
@@ -19,11 +19,20 @@
   <xacro:arg name="multiple" default="false"/>
   <xacro:property name="is_multiple" value="$(arg multiple)" />
+  <!-- ROS 2 Control-->
+  <xacro:include filename="$(find talos_description)/ros2_control/ros2_control.urdf.xacro" />
+  <xacro:talos_ros2_control use_sim="$(arg use_sim)"/>
   <!--************************-->
   <!--        BASE_LINK       -->
   <!--************************-->
+  <link name="world"/>
+  <joint name="world_fixed" type="fixed">
+      <origin xyz="0 0 0" rpy="0 0 0"/>
+      <parent link="world"/>
+      <child link="base_link"/>
+  </joint>
   <link name="base_link">
     <inertial>
       <origin xyz="-0.08222 0.00838 -0.07261" rpy="0.00000 0.00000 0.00000"/>
-      <mass value="13.53810"/>
+      <mass value="13.503810"/>
       <inertia ixx="0.06989000000" ixy="-0.00011700000" ixz="0.00023000000"
                iyy="0.03998200000" iyz="-0.00132500000"
@@ -52,6 +61,3 @@
   <!-- Materials for visualization -->
   <xacro:include filename="$(find talos_description)/urdf/materials.urdf.xacro" />
-  <!-- ROS 2 Control-->
-  <xacro:include filename="$(find talos_description)/ros2_control/ros2_control.urdf.xacro" />
-  <xacro:talos_ros2_control use_sim="$(arg use_sim)"/>
 </robot>

File: talos_description/ros2_control/ros2_control.urdf.xacro (robot description, xacro)
@@ -21,7 +21,7 @@
     <xacro:include filename="$(find talos_description)/urdf/head/head.ros2_control.xacro" />
     <xacro:include filename="$(find talos_description)/urdf/leg/leg.ros2_control.xacro" />
+    <xacro:include filename="$(find talos_description)/urdf/torso/torso.ros2_control.xacro" />
     <!-- Calibration offsets -->
     <xacro:include filename="$(find talos_description_calibration)/urdf/calibration/calibration_constants.urdf.xacro" />
-    <xacro:property name="leg_reduction"    value="1.0" /><!-- i don't like here-->
     <ros2_control name="ros2_control_talos_system" type="system">
       <hardware>
@@ -33,8 +33,8 @@
         </xacro:unless>
       </hardware>
-      <!-- IMU -->
+      <!-- IMU
       <xacro:if value="$(arg use_sim)">
         <xacro:ros2_control_imu name="base_imu_sensor"/>
-      </xacro:if>
+      </xacro:if>-->
       <!-- arm right-->
       <xacro:ros2_control_arm name="arm" side="right" number="1"/>
@@ -60,24 +60,25 @@
       <xacro:ros2_control_gripper name="gripper_left"/>
       <!-- Head -->
-      <xacro:ros2_control_head name="head" offset_value_1="${head_1_joint_yaw_offset}" offset_value_2="${head_2_joint_yaw_offset}"/>
+      <xacro:ros2_control_head name="head" number_1="1" number_2="2" offset_value_1="${head_1_joint_yaw_offset}" offset_value_2="${head_2_joint_yaw_offset}"/>
       <!-- Torso -->
-      <xacro:ros2_control_torso name="torso"/>
+      <xacro:ros2_control_torso name="torso" number="1"/>
+      <xacro:ros2_control_torso name="torso" number="2"/>
        <!-- Force Torque sensor-->
-      <xacro:ros2_control_force_torque_sensor name="wrist_right_ft_sensor"/>
-      <xacro:ros2_control_force_torque_sensor name="wrist_left_ft_sensor"/>
+      <!-- <xacro:ros2_control_force_torque_sensor name="wrist_right_ft_sensor"/>
+      <xacro:ros2_control_force_torque_sensor name="wrist_left_ft_sensor"/> -->
       <!-- Leg left -->
-      <xacro:ros2_control_leg side="left" number="1" leg_reduction="${leg_reduction}" />
-      <xacro:ros2_control_leg side="left" number="2" leg_reduction="${leg_reduction}" />
-      <xacro:ros2_control_leg side="left" number="3" leg_reduction="${leg_reduction}" />
-      <xacro:ros2_control_leg side="left" number="4" leg_reduction="${leg_reduction}" />
-      <xacro:ros2_control_leg side="left" number="5" leg_reduction="${leg_reduction}" />
-      <xacro:ros2_control_leg side="left" number="6" leg_reduction="${leg_reduction}" />
+      <xacro:ros2_control_leg side="left" number="1" />
+      <xacro:ros2_control_leg side="left" number="2" />
+      <xacro:ros2_control_leg side="left" number="3" />
+      <xacro:ros2_control_leg side="left" number="4" />
+      <xacro:ros2_control_leg side="left" number="5" />
+      <xacro:ros2_control_leg side="left" number="6" />
       <!-- Leg right -->
-      <xacro:ros2_control_leg side="right" number="1" leg_reduction="${leg_reduction}" />
-      <xacro:ros2_control_leg side="right" number="2" leg_reduction="${leg_reduction}" />
-      <xacro:ros2_control_leg side="right" number="3" leg_reduction="${leg_reduction}" />
-      <xacro:ros2_control_leg side="right" number="4" leg_reduction="${leg_reduction}" />
-      <xacro:ros2_control_leg side="right" number="5" leg_reduction="${leg_reduction}" />
-      <xacro:ros2_control_leg side="right" number="6" leg_reduction="${leg_reduction}" />
+      <xacro:ros2_control_leg side="right" number="1" />
+      <xacro:ros2_control_leg side="right" number="2" />
+      <xacro:ros2_control_leg side="right" number="3" />
+      <xacro:ros2_control_leg side="right" number="4" />
+      <xacro:ros2_control_leg side="right" number="5" />
+      <xacro:ros2_control_leg side="right" number="6" />
     </ros2_control>
   </xacro:macro>

File: talos_description/urdf/gripper/gripper.ros2_control.xacro (robot description, xacro)
@@ -22,4 +22,64 @@
       <state_interface name="effort" />
     </joint>
+    <joint name="${name}_inner_double_joint">
+      <param name="mimic">${name}_joint</param>
+      <param name="multiplier">1</param>
+      <command_interface name="position" />
+      <command_interface name="velocity" />
+      <command_interface name="effort" />
+      <state_interface name="position" />
+      <state_interface name="velocity" />
+      <state_interface name="effort" />
+    </joint>
+    <joint name="${name}_fingertip_1_joint">
+      <param name="mimic">${name}_joint</param>
+      <param name="multiplier">1</param>
+      <command_interface name="position" />
+      <command_interface name="velocity" />
+      <command_interface name="effort" />
+      <state_interface name="position" />
+      <state_interface name="velocity" />
+      <state_interface name="effort" />
+    </joint>
+    <joint name="${name}_fingertip_2_joint">
+      <param name="mimic">${name}_joint</param>
+      <param name="multiplier">1</param>
+      <command_interface name="position" />
+      <command_interface name="velocity" />
+      <command_interface name="effort" />
+      <state_interface name="position" />
+      <state_interface name="velocity" />
+      <state_interface name="effort" />
+    </joint>
+    <joint name="${name}_motor_single_joint">
+      <param name="mimic">${name}_joint</param>
+      <param name="multiplier">-1</param>
+      <command_interface name="position" />
+      <command_interface name="velocity" />
+      <command_interface name="effort" />
+      <state_interface name="position" />
+      <state_interface name="velocity" />
+      <state_interface name="effort" />
+    </joint>
+    <joint name="${name}_inner_single_joint">
+      <param name="mimic">${name}_joint</param>
+      <param name="multiplier">-1</param>
+      <command_interface name="position" />
+      <command_interface name="velocity" />
+      <command_interface name="effort" />
+      <state_interface name="position" />
+      <state_interface name="velocity" />
+      <state_interface name="effort" />
+    </joint>
+    <joint name="${name}_fingertip_3_joint">
+      <param name="mimic">${name}_joint</param>
+      <param name="multiplier">-1</param>
+      <command_interface name="position" />
+      <command_interface name="velocity" />
+      <command_interface name="effort" />
+      <state_interface name="position" />
+      <state_interface name="velocity" />
+      <state_interface name="effort" />
+    </joint>
    <!-- transmissions -->
   <xacro:include filename="$(find talos_description)/urdf/gripper/gripper.transmission.xacro" />

File: talos_description/urdf/head/head.ros2_control.xacro (robot description, xacro)
@@ -13,6 +13,6 @@
  -->
 <robot xmlns:xacro="http://ros.org/wiki/xacro">
-  <xacro:macro name="ros2_control_head" params="name offset_value_1 offset_value_2" >
-    <joint name="${name}_1_joint">
+  <xacro:macro name="ros2_control_head" params="name number_1 number_2 offset_value_1 offset_value_2" >
+    <joint name="${name}_${number_1}_joint">
       <command_interface name="position" />
       <command_interface name="velocity" />
@@ -22,5 +22,5 @@
       <state_interface name="effort" />
     </joint>
-    <joint name="${name}_2_joint">
+    <joint name="${name}_${number_2}_joint">
       <command_interface name="position" />
       <command_interface name="velocity" />
@@ -32,5 +32,5 @@
     <!-- Transmission -->
     <xacro:include filename="$(find talos_description)/urdf/head/head.transmission.xacro" />
-    <xacro:talos_head_differential_transmission name="${name}" number1="1" number2="2"
+    <xacro:talos_head_differential_transmission name="${name}" number1="${number_1}" number2="${number_2}"
                                                 act_reduction1="1.0" act_reduction2="1.0"
                                                 jnt_reduction1="1.0" jnt_reduction2="2.0"

File: talos_description/urdf/leg/leg.ros2_control.xacro (robot description, xacro)
@@ -13,5 +13,5 @@
  -->
 <robot xmlns:xacro="http://ros.org/wiki/xacro">
-  <xacro:macro name="ros2_control_leg" params="side number leg_reduction flexibility:=false" >
+  <xacro:macro name="ros2_control_leg" params="side number leg_reduction:=1.0 flexibility:=false" >
     <joint name="leg_${side}_${number}_joint">
       <command_interface name="position" />

File: talos_description/urdf/torso/torso.ros2_control.xacro (robot description, xacro)
@@ -13,6 +13,6 @@
  -->
 <robot xmlns:xacro="http://ros.org/wiki/xacro">
-  <xacro:macro name="ros2_control_torso" params="name" >
-    <joint name="${name}_1_joint">
+  <xacro:macro name="ros2_control_torso" params="name number" >
+    <joint name="${name}_${number}_joint">
       <command_interface name="position" />
       <command_interface name="velocity" />
@@ -22,15 +22,7 @@
       <state_interface name="effort" />
     </joint>
-    <joint name="${name}_2_joint">
-      <command_interface name="position" />
-      <command_interface name="velocity" />
-      <command_interface name="effort" />
-      <state_interface name="position" />
-      <state_interface name="velocity" />
-      <state_interface name="effort" />
-    </joint>
-   <!-- transmissions -->
-  <xacro:include filename="$(find talos_description)/urdf/torso/torso.transmission.xacro" />
-  <xacro:talos_torso_differential_transmission name="${name}" number1="1" number2="2"
+    <!-- transmissions -->
+    <xacro:include filename="$(find talos_description)/urdf/torso/torso.transmission.xacro" />
+    <xacro:talos_torso_differential_transmission name="${name}" number1="1" number2="2"
                                                 act_reduction1="1.0" act_reduction2="1.0"
                                                 jnt_reduction1="1.0" jnt_reduction2="1.0" />

File: talos_description/urdf/torso/torso.urdf.xacro (robot description, xacro)
@@ -17,4 +17,11 @@
     <xacro:include filename="$(find talos_description)/test/calibration/calibration_constants.urdf.xacro" />
   </xacro:if>
+  <!-- Fixed world frame -->
+  <link name="world"/>
+  <joint name="world_fixed" type="fixed">
+      <origin xyz="0 0 0" rpy="0 0 0"/>
+      <parent link="world"/>
+      <child link="base_link"/>
+  </joint>
  <!--Constant parameters-->
   <xacro:property name="torso_max_vel"  value="5.4" />

File: talos_description_inertial/urdf/inertial.xacro (robot description, xacro)
@@ -257,5 +257,5 @@
       <mass value="2.235009"/>
       <inertia ixx="0.01049849" ixy="0.00004097" ixz="0.00009771" iyy="0.00534086" iyz="-0.0011949" izz="0.00708595" />
-      <origin rpy="0 0 0" xyz="0.08472839 -0.10997434 0.01705898"/>
+      <origin rpy="0 0 0" xyz="0.08472839 0.10997434 0.01705898"/>
     </inertial>
   </xacro:macro>
