Commit message: fix inertia signs leg_left_1_link and arm_right_4_link_inertial

File: talos_description_inertial/urdf/inertial.xacro (robot description, xacro)
@@ -82,5 +82,5 @@
       <mass value="0.815675"/>
       <inertia ixx="0.00299913" ixy="-0.00009333" ixz="0.0003389" iyy="0.00303994" iyz="-0.0004233" izz="0.00126248" />
-      <origin rpy="0 0 0" xyz="-0.00810404 -0.01944328 -0.03329237"/>
+      <origin rpy="0 0 0" xyz="-0.00810404 0.01944328 -0.03329237"/>
     </inertial>
   </xacro:macro>
@@ -257,5 +257,5 @@
       <mass value="2.235009"/>
       <inertia ixx="0.01049849" ixy="0.00004097" ixz="0.00009771" iyy="0.00534086" iyz="-0.0011949" izz="0.00708595" />
-      <origin rpy="0 0 0" xyz="0.08472839 -0.10997434 0.01705898"/>
+      <origin rpy="0 0 0" xyz="0.08472839 0.10997434 0.01705898"/>
     </inertial>
   </xacro:macro>

Commit message: update inertia signs

File: talos_description_inertial/urdf/inertial.xacro (robot description, xacro)
@@ -81,5 +81,5 @@
     <inertial>
       <mass value="0.815675"/>
-      <inertia ixx="0.00299913" ixy="-0.00009333" ixz="0.0003389" iyy="0.00303994" iyz="-0.0004233" izz="0.00126248" />
+      <inertia ixx="0.00299913" ixy="0.00009333" ixz="0.0003389" iyy="0.00303994" iyz="0.0004233" izz="0.00126248" />
       <origin rpy="0 0 0" xyz="-0.00810404 0.01944328 -0.03329237"/>
     </inertial>
@@ -256,5 +256,5 @@
     <inertial>
       <mass value="2.235009"/>
-      <inertia ixx="0.01049849" ixy="0.00004097" ixz="0.00009771" iyy="0.00534086" iyz="-0.0011949" izz="0.00708595" />
+      <inertia ixx="0.01049849" ixy="-0.00004097" ixz="0.00009771" iyy="0.00534086" iyz="0.0011949" izz="0.00708595" />
       <origin rpy="0 0 0" xyz="0.08472839 0.10997434 0.01705898"/>
     </inertial>

Commit message: update inertia signs

File: talos_description_inertial/urdf/inertial.xacro (robot description, xacro)
@@ -81,6 +81,6 @@
     <inertial>
       <mass value="0.815675"/>
-      <inertia ixx="0.00299913" ixy="-0.00009333" ixz="0.0003389" iyy="0.00303994" iyz="-0.0004233" izz="0.00126248" />
-      <origin rpy="0 0 0" xyz="-0.00810404 -0.01944328 -0.03329237"/>
+      <inertia ixx="0.00299913" ixy="0.00009333" ixz="0.0003389" iyy="0.00303994" iyz="0.0004233" izz="0.00126248" />
+      <origin rpy="0 0 0" xyz="-0.00810404 0.01944328 -0.03329237"/>
     </inertial>
   </xacro:macro>
@@ -256,5 +256,5 @@
     <inertial>
       <mass value="2.235009"/>
-      <inertia ixx="0.01049849" ixy="0.00004097" ixz="0.00009771" iyy="0.00534086" iyz="-0.0011949" izz="0.00708595" />
+      <inertia ixx="0.01049849" ixy="-0.00004097" ixz="0.00009771" iyy="0.00534086" iyz="0.0011949" izz="0.00708595" />
       <origin rpy="0 0 0" xyz="0.08472839 0.10997434 0.01705898"/>
     </inertial>
