Commit message: update gripper mimic joint and sensors

File: talos_description/gazebo/gazebo.urdf.xacro (robot description, xacro)
@@ -39,5 +39,5 @@
     <!--- backwards compatibility, used to be gazebo_world_odometry pal plugin-->
     <plugin filename="libgazebo_ros_p3d.so" name="gazebo_ros_odometry">
-      <body_name>base_footprint</body_name>
+      <body_name>base_footprint</body_name><!--base_footprint-->
       <always_on>true</always_on>
       <update_rate>1000.0</update_rate>
@@ -50,4 +50,5 @@
     </plugin>
   </gazebo>
+<!-- TODO
   <gazebo>
     <plugin filename="libgazebo_ros_force.so" name="gazebo_ros_force">
@@ -56,8 +57,6 @@
     </plugin>
   </gazebo>
+-->
   <gazebo reference="imu_link">
-    <!-- this is expected to be reparented to pelvis with appropriate offset
-         when imu_link is reduced by fixed joint reduction -->
-    <!-- todo: this is working with gazebo 1.4, need to write a unit test -->
     <sensor name="imu_sensor" type="imu">
       <always_on>1</always_on>
@@ -66,34 +65,4 @@
         <noise>
           <type>gaussian</type>
-          <!-- Noise parameters from Boston Dynamics
-               (http://gazebosim.org/wiki/Sensor_noise):
-                 rates (rad/s): mean=0, stddev=2e-4
-                 accels (m/s/s): mean=0, stddev=1.7e-2
-                 rate bias (rad/s): 5e-6 - 1e-5
-                 accel bias (m/s/s): 1e-1
-               Experimentally, simulation provide rates with noise of
-               about 1e-3 rad/s and accels with noise of about 1e-1 m/s/s.
-               So we don't expect to see the noise unless number of inner iterations
-               are increased.
-               We will add bias.  In this model, bias is sampled once for rates
-               and once for accels at startup; the sign (negative or positive)
-               of each bias is then switched with equal probability.  Thereafter,
-               the biases are fixed additive offsets.  We choose
-               bias means and stddevs to produce biases close to the provided
-               data. -->
-          <!--
-          <rate>
-            <mean>0.0</mean>
-            <stddev>2e-4</stddev>
-            <bias_mean>0.0000075</bias_mean>
-            <bias_stddev>0.0000008</bias_stddev>
-          </rate>
-          <accel>
-            <mean>0.0</mean>
-            <stddev>1.7e-2</stddev>
-            <bias_mean>0.1</bias_mean>
-            <bias_stddev>0.001</bias_stddev>
-          </accel>
-          -->
           <rate>
             <mean>0.0</mean>
@@ -110,13 +79,5 @@
         </noise>
       </imu>
-      <plugin name="base_imu" filename="libgazebo_ros_imu_sensor.so">
-        <ros>
-          <!-- publish to /imu/data -->
-          <remapping>~/out:=base_imu</remapping>
-        </ros>
-      </plugin>
     </sensor>
   </gazebo>
-  <!-- define global properties -->
-  <!-- <xacro:property name="M_PI" value="3.1415926535897931" /> -->
 </robot>

File: talos_description/ros2_control/ros2_control.urdf.xacro (robot description, xacro)
@@ -36,5 +36,5 @@
       <!-- IMU -->
       <xacro:if value="$(arg use_sim)">
-        <xacro:ros2_control_imu name="base_imu_sensor"/>
+        <xacro:ros2_control_imu name="imu_sensor"/>
       </xacro:if>
       <!-- arm right-->

File: talos_description/urdf/gripper/gripper.ros2_control.xacro (robot description, xacro)
@@ -14,4 +14,16 @@
 <robot xmlns:xacro="http://ros.org/wiki/xacro">
   <xacro:macro name="ros2_control_gripper" params="name" >
+    <xacro:macro name="ros2_control_talos_gripper_mimic_joint" params="mimic_joint_name actuated_joint_name multiplier" >
+      <joint name="${mimic_joint_name}">
+        <param name="mimic">${actuated_joint_name}</param>
+        <param name="multiplier">${multiplier}</param>
+        <command_interface name="position" />
+        <command_interface name="velocity" />
+        <command_interface name="effort" />
+        <state_interface name="position"/>
+        <state_interface name="velocity" />
+        <state_interface name="effort" />
+      </joint>
+    </xacro:macro>
     <joint name="${name}_joint">
       <command_interface name="position" />
@@ -22,64 +34,22 @@
       <state_interface name="effort" />
     </joint>
-    <joint name="${name}_inner_double_joint">
-      <param name="mimic">${name}_joint</param>
-      <param name="multiplier">1</param>
-      <command_interface name="position" />
-      <command_interface name="velocity" />
-      <command_interface name="effort" />
-      <state_interface name="position" />
-      <state_interface name="velocity" />
-      <state_interface name="effort" />
-    </joint>
-    <joint name="${name}_fingertip_1_joint">
-      <param name="mimic">${name}_joint</param>
-      <param name="multiplier">1</param>
-      <command_interface name="position" />
-      <command_interface name="velocity" />
-      <command_interface name="effort" />
-      <state_interface name="position" />
-      <state_interface name="velocity" />
-      <state_interface name="effort" />
-    </joint>
-    <joint name="${name}_fingertip_2_joint">
-      <param name="mimic">${name}_joint</param>
-      <param name="multiplier">1</param>
-      <command_interface name="position" />
-      <command_interface name="velocity" />
-      <command_interface name="effort" />
-      <state_interface name="position" />
-      <state_interface name="velocity" />
-      <state_interface name="effort" />
-    </joint>
-    <joint name="${name}_motor_single_joint">
-      <param name="mimic">${name}_joint</param>
-      <param name="multiplier">-1</param>
-      <command_interface name="position" />
-      <command_interface name="velocity" />
-      <command_interface name="effort" />
-      <state_interface name="position" />
-      <state_interface name="velocity" />
-      <state_interface name="effort" />
-    </joint>
-    <joint name="${name}_inner_single_joint">
-      <param name="mimic">${name}_joint</param>
-      <param name="multiplier">-1</param>
-      <command_interface name="position" />
-      <command_interface name="velocity" />
-      <command_interface name="effort" />
-      <state_interface name="position" />
-      <state_interface name="velocity" />
-      <state_interface name="effort" />
-    </joint>
-    <joint name="${name}_fingertip_3_joint">
-      <param name="mimic">${name}_joint</param>
-      <param name="multiplier">-1</param>
-      <command_interface name="position" />
-      <command_interface name="velocity" />
-      <command_interface name="effort" />
-      <state_interface name="position" />
-      <state_interface name="velocity" />
-      <state_interface name="effort" />
-    </joint>
+    <xacro:ros2_control_talos_gripper_mimic_joint mimic_joint_name="${name}_inner_double_joint"
+                                                    actuated_joint_name="${name}_joint"
+                                                    multiplier="1"/>
+    <xacro:ros2_control_talos_gripper_mimic_joint mimic_joint_name="${name}_fingertip_1_joint"
+                                                    actuated_joint_name="${name}_joint"
+                                                    multiplier="1"/>
+    <xacro:ros2_control_talos_gripper_mimic_joint mimic_joint_name="${name}_fingertip_2_joint"
+                                                    actuated_joint_name="${name}_joint"
+                                                    multiplier="1"/>
+    <xacro:ros2_control_talos_gripper_mimic_joint mimic_joint_name="${name}_motor_single_joint"
+                                                    actuated_joint_name="${name}_joint"
+                                                    multiplier="-1"/>
+    <xacro:ros2_control_talos_gripper_mimic_joint mimic_joint_name="${name}_inner_single_joint"
+                                                    actuated_joint_name="${name}_joint"
+                                                    multiplier="-1"/>
+    <xacro:ros2_control_talos_gripper_mimic_joint mimic_joint_name="${name}_fingertip_3_joint"
+                                                    actuated_joint_name="${name}_joint"
+                                                    multiplier="-1"/>
    <!-- transmissions -->
   <xacro:include filename="$(find talos_description)/urdf/gripper/gripper.transmission.xacro" />

File: talos_description/urdf/gripper/gripper.urdf.xacro (robot description, xacro)
@@ -1,8 +1,21 @@
 <?xml version="1.0"?>
 <robot xmlns:xacro="http://ros.org/wiki/xacro">
-  <!--File includes-->
   <xacro:include filename="$(find talos_description)/urdf/deg_to_rad.xacro" />
-  <xacro:include filename="$(find talos_description)/urdf/gripper/gripper.gazebo.xacro" />
   <xacro:macro name="talos_gripper" params="name parent reflect">
+            <xacro:macro name="dummy_mimic_joint" params="name parent">
+              <link name="${name}_dummy_mimic_link"/>
+              <joint name="${name}_joint_mimic" type="fixed">
+                <parent link="${parent}" />
+                <child link="${name}_dummy_mimic_link" />
+              </joint>
+            </xacro:macro>
+            <xacro:macro name="finger_mimic_dummy" params="name">
+              <xacro:dummy_mimic_joint name="${name}_fingertip_1" parent="${name}_base_link"/>
+              <xacro:dummy_mimic_joint name="${name}_fingertip_2" parent="${name}_base_link"/>
+              <xacro:dummy_mimic_joint name="${name}_inner_single" parent="${name}_base_link"/>
+              <xacro:dummy_mimic_joint name="${name}_fingertip_3" parent="${name}_base_link"/>
+              <xacro:dummy_mimic_joint name="${name}_motor_single" parent="${name}_base_link"/>
+              <xacro:dummy_mimic_joint name="${name}_inner_double" parent="${name}_base_link"/>
+            </xacro:macro>
             <link name="${name}_base_link">
               <xacro:call macro="${name}_base_link_inertial" />
@@ -203,12 +216,55 @@
               <mimic joint="${name}_joint" multiplier="${-1.0}" offset="0.0" />
             </joint>
-        <xacro:virtual_joints name="${name}" />
-        <!-- virtual mimic joints -->
-<!--         <xacro:gripper_virtual_transmission name="${name}_inner_double" reduction="1.0"/>
-        <xacro:gripper_virtual_transmission name="${name}_fingertip_1" reduction="1.0"/>
-        <xacro:gripper_virtual_transmission name="${name}_fingertip_2" reduction="1.0"/>
-        <xacro:gripper_virtual_transmission name="${name}_inner_single" reduction="1.0"/>
-        <xacro:gripper_virtual_transmission name="${name}_motor_single" reduction="1.0"/>
-        <xacro:gripper_virtual_transmission name="${name}_fingertip_3" reduction="1.0"/> -->
+            <gazebo reference="${name}_joint">
+                <implicitSpringDamper>1</implicitSpringDamper>
+                <provideFeedback>1</provideFeedback>
+              </gazebo>
+              <gazebo reference="${name}_inner_double_joint">
+                <implicitSpringDamper>1</implicitSpringDamper>
+                <provideFeedback>1</provideFeedback>
+              </gazebo>
+              <gazebo reference="${name}_fingertip_1_joint">
+                <implicitSpringDamper>1</implicitSpringDamper>
+                <provideFeedback>1</provideFeedback>
+              </gazebo>
+              <gazebo reference="${name}_fingertip_2_joint">
+                <implicitSpringDamper>1</implicitSpringDamper>
+                <provideFeedback>1</provideFeedback>
+              </gazebo>
+              <gazebo reference="${name}_motor_single_joint">
+                <implicitSpringDamper>1</implicitSpringDamper>
+                <provideFeedback>1</provideFeedback>
+              </gazebo>
+              <gazebo reference="${name}_fingertip_3_joint">
+                <implicitSpringDamper>1</implicitSpringDamper>
+                <provideFeedback>1</provideFeedback>
+              </gazebo>
+              <gazebo reference="${name}_base_link">
+                <material>Gazebo/FlatBlack</material>
+              </gazebo>
+              <gazebo reference="${name}_motor_double_link">
+                <material>Gazebo/Orange</material>
+              </gazebo>
+              <gazebo reference="${name}_inner_double_link">
+                <material>Gazebo/Orange</material>
+              </gazebo>
+              <gazebo reference="${name}_fingertip_1_link">
+                <material>Gazebo/FlatBlack</material>
+              </gazebo>
+              <gazebo reference="${name}_motor_single_link">
+                <material>Gazebo/Orange</material>
+              </gazebo>
+              <gazebo reference="${name}_inner_single_link">
+                <material>Gazebo/Orange</material>
+              </gazebo>
+              <gazebo reference="${name}_fingertip_2_link">
+                <material>Gazebo/FlatBlack</material>
+              </gazebo>
+              <gazebo reference="${name}_fingertip_3_link">
+                <material>Gazebo/FlatBlack</material>
+              </gazebo>
+              <!-- Temporary fix until mimic joint works properly with MoveIt!-->
+              <xacro:finger_mimic_dummy name="${name}"/>
+              <xacro:dummy_mimic_joint name="${name}_link" parent="${name}_base_link"/>
   </xacro:macro>
 </robot>

File: talos_description/urdf/talos_full_common.urdf.xacro (robot description, xacro)
@@ -18,4 +18,5 @@
   <xacro:include filename="$(find talos_description)/urdf/arm/arm.urdf.xacro" />
   <xacro:include filename="$(find talos_description)/urdf/sensors/ftsensor.urdf.xacro" />
+  <xacro:include filename="$(find talos_description)/urdf/sensors/ftsensor.gazebo.xacro" />
   <xacro:include filename="$(find talos_description)/urdf/gripper/gripper.urdf.xacro" />
   <xacro:include filename="$(find talos_description)/urdf/leg/leg.urdf.xacro" />
@@ -35,4 +36,6 @@
   <xacro:ft_sensor name="wrist" parent="arm_right_7_link" side="right" reflect="1"  />
   <xacro:ft_sensor name="wrist" parent="arm_left_7_link"  side="left"  reflect="-1" />
+  <xacro:force_torque_sensor_gazebo name="wrist_left_ft" update_rate="100"/>
+  <xacro:force_torque_sensor_gazebo name="wrist_right_ft" update_rate="100"/>
   <xacro:talos_gripper name="gripper_left" parent="wrist_left_ft_tool_link" reflect="1" />
   <xacro:talos_gripper name="gripper_right" parent="wrist_right_ft_tool_link" reflect="-1" />

Commit message: [talos_descirption] Try to add the force sensors at the feet

File: talos_description/gazebo/gazebo.urdf.xacro (robot description, xacro)
@@ -13,38 +13,24 @@
  -->
 <robot name="talos" xmlns:xacro="http://ros.org/wiki/xacro">
-  <gazebo>
-    <plugin filename="libgazebo_ros2_control.so" name="gazebo_ros2_control">
-      <!-- in the future move this param file somewhere else -->
-      <parameters>$(find talos_controller_configuration)/config/gazebo_controller_manager_cfg.yaml</parameters>
-      <xacro:if value="${is_multiple}">
-        <!-- Do something about multirobot -->
-      </xacro:if>
-      <xacro:unless value="${is_multiple}">
-        <!-- Do something about multirobot -->
-      </xacro:unless>
-    </plugin>
-  </gazebo>
-  <gazebo reference="imu_link">
-    <sensor name="imu_sensor" type="imu">
-      <always_on>1</always_on>
-      <update_rate>1000.0</update_rate>
-      <imu>
-        <noise>
-          <type>gaussian</type>
-          <rate>
-            <mean>0.0</mean>
-            <stddev>0.0</stddev>
-            <bias_mean>0.000000</bias_mean>
-            <bias_stddev>0.0000008</bias_stddev>
-          </rate>
-          <accel>
-            <mean>0.0</mean>
-            <stddev>0.0</stddev>
-            <bias_mean>0.0</bias_mean>
-            <bias_stddev>0.000</bias_stddev>
-          </accel>
-        </noise>
-      </imu>
-    </sensor>
-  </gazebo>
+  <xacro:include filename="$(find talos_description)/urdf/sensors/imu.gazebo.xacro" />
+  <xacro:include filename="$(find talos_description)/urdf/sensors/ftsensor.gazebo.xacro" />
+  <xacro:macro name="talos_gazebo">
+    <gazebo>
+      <plugin filename="libgazebo_ros2_control.so" name="gazebo_ros2_control">
+        <!-- in the future move this param file somewhere else -->
+        <parameters>$(find talos_controller_configuration)/config/gazebo_controller_manager_cfg.yaml</parameters>
+        <xacro:if value="${is_multiple}">
+          <!-- Do something about multirobot -->
+        </xacro:if>
+        <xacro:unless value="${is_multiple}">
+          <!-- Do something about multirobot -->
+        </xacro:unless>
+      </plugin>
+    </gazebo>
+    <xacro:imu_sensor_gazebo update_rate="1000.0"/>
+    <xacro:force_torque_sensor_gazebo name="wrist_left_ft" update_rate="1000.0"/>
+    <xacro:force_torque_sensor_gazebo name="wrist_right_ft" update_rate="1000.0"/>
+    <!-- <xacro:force_torque_sensor_gazebo name="ankle_left_ft" update_rate="1000.0"/>
+    <xacro:force_torque_sensor_gazebo name="ankle_right_ft" update_rate="1000.0"/> -->
+  </xacro:macro>
 </robot>

File: talos_description/ros2_control/ros2_control.urdf.xacro (robot description, xacro)
@@ -15,5 +15,4 @@
        name="talos" >
   <xacro:macro name="talos_ros2_control" params="use_sim:=^|false">
-    <xacro:include filename="$(find talos_description)/urdf/sensors/ftsensor.ros2_control.xacro" />
     <xacro:include filename="$(find talos_description)/urdf/arm/arm.ros2_control.xacro" />
     <xacro:include filename="$(find talos_description)/urdf/arm/wrist.ros2_control.xacro"/>
@@ -22,5 +21,6 @@
     <xacro:include filename="$(find talos_description)/urdf/leg/leg.ros2_control.xacro" />
     <xacro:include filename="$(find talos_description)/urdf/torso/torso.ros2_control.xacro" />
-    <xacro:include filename="$(find talos_description)/urdf/sensors/imusensor.ros2_control.xacro" />
+    <xacro:include filename="$(find talos_description)/urdf/sensors/imu.ros2_control.xacro" />
+    <xacro:include filename="$(find talos_description)/urdf/sensors/ftsensor.ros2_control.xacro" />
     <!-- Calibration offsets -->
     <xacro:include filename="$(find talos_description_calibration)/urdf/calibration/calibration_constants.urdf.xacro" />
@@ -65,7 +65,9 @@
       <xacro:ros2_control_torso name="torso" number="1"/>
       <xacro:ros2_control_torso name="torso" number="2"/>
-       <!-- Force Torque sensor-->
+      <!-- Force Torque sensor-->
       <xacro:ros2_control_force_torque_sensor name="wrist_right_ft_sensor"/>
       <xacro:ros2_control_force_torque_sensor name="wrist_left_ft_sensor"/>
+      <xacro:ros2_control_force_torque_sensor name="ankle_right_ft_sensor"/>
+      <xacro:ros2_control_force_torque_sensor name="ankle_left_ft_sensor"/>
       <!-- Leg left -->
       <xacro:ros2_control_leg side="left" number="1" />

File: talos_description/urdf/sensors/ftsensor.gazebo.xacro (robot description, xacro)
@@ -14,15 +14,15 @@
 <robot xmlns:xacro="http://ros.org/wiki/xacro">
   <xacro:macro name="force_torque_sensor_gazebo" params="name update_rate">
-  <gazebo reference="${name}_joint">
-    <preserveFixedJoint>true</preserveFixedJoint> <!-- in case this is in a fixed joint -->
-    <sensor name="${name}_sensor" type="force_torque">
-      <update_rate>${update_rate}</update_rate>
-      <visualize>true</visualize>
-      <force_torque>
-        <frame>child</frame>
-        <measure_direction>child_to_parent</measure_direction>
-      </force_torque>
-    </sensor>
-</gazebo>
-</xacro:macro>
+    <gazebo reference="${name}_joint">
+      <preserveFixedJoint>true</preserveFixedJoint> <!-- in case this is in a fixed joint -->
+      <sensor name="${name}_sensor" type="force_torque">
+        <update_rate>${update_rate}</update_rate>
+        <visualize>true</visualize>
+        <force_torque>
+          <frame>child</frame>
+          <measure_direction>child_to_parent</measure_direction>
+        </force_torque>
+      </sensor>
+    </gazebo>
+  </xacro:macro>
 </robot>

File: talos_description/urdf/talos_full_common.urdf.xacro (robot description, xacro)
@@ -18,5 +18,4 @@
   <xacro:include filename="$(find talos_description)/urdf/arm/arm.urdf.xacro" />
   <xacro:include filename="$(find talos_description)/urdf/sensors/ftsensor.urdf.xacro" />
-  <xacro:include filename="$(find talos_description)/urdf/sensors/ftsensor.gazebo.xacro" />
   <xacro:include filename="$(find talos_description)/urdf/gripper/gripper.urdf.xacro" />
   <xacro:include filename="$(find talos_description)/urdf/leg/leg.urdf.xacro" />
@@ -24,4 +23,9 @@
   <xacro:include filename="$(find talos_description_inertial)/urdf/inertial.xacro" />
   <xacro:include filename="$(find talos_description)/urdf/extras/addons.urdf.xacro" />
+  <xacro:include filename="$(find talos_description)/ros2_control/ros2_control.urdf.xacro" />
+  <!-- Generic simulator_gazebo plugins -->
+  <xacro:include filename="$(find talos_description)/gazebo/gazebo.urdf.xacro" />
+  <!-- Materials for visualization -->
+  <xacro:include filename="$(find talos_description)/urdf/materials.urdf.xacro" />
   <xacro:talos_torso name="torso" />
   <xacro:if value="$(arg enable_crane)">
@@ -36,18 +40,11 @@
   <xacro:ft_sensor name="wrist" parent="arm_right_7_link" side="right" reflect="1"  />
   <xacro:ft_sensor name="wrist" parent="arm_left_7_link"  side="left"  reflect="-1" />
-  <xacro:force_torque_sensor_gazebo name="wrist_left_ft" update_rate="100"/>
-  <xacro:force_torque_sensor_gazebo name="wrist_right_ft" update_rate="100"/>
   <xacro:talos_gripper name="gripper_left" parent="wrist_left_ft_tool_link" reflect="1" />
   <xacro:talos_gripper name="gripper_right" parent="wrist_right_ft_tool_link" reflect="-1" />
   <xacro:talos_leg prefix="left"  reflect="1" flexibility="$(arg flexibility)"/>
   <xacro:talos_leg prefix="right" reflect="-1" flexibility="$(arg flexibility)"/>
-  <!-- Macro to have the add-on links specific to each TALOS -->
-  <xacro:talos_addons />
-  <!-- Generic simulator_gazebo plugins -->
-  <xacro:include filename="$(find talos_description)/gazebo/gazebo.urdf.xacro" />
-  <!-- Materials for visualization -->
-  <xacro:include filename="$(find talos_description)/urdf/materials.urdf.xacro" />
-  <!-- ROS 2 Control-->
-  <xacro:include filename="$(find talos_description)/ros2_control/ros2_control.urdf.xacro" />
+  <xacro:talos_addons/>
+  <xacro:talos_gazebo/>
+  <xacro:talos_materials/>
   <xacro:talos_ros2_control use_sim="$(arg use_sim)"/>
 </robot>
