Commit message: Try to add the ankle FT sensors for Talos and connect them to ros2_control

File: talos_description/gazebo/gazebo.urdf.xacro (robot description, xacro)
@@ -31,6 +31,6 @@
     <xacro:force_torque_sensor_gazebo name="wrist_left_ft" update_rate="1000.0"/>
     <xacro:force_torque_sensor_gazebo name="wrist_right_ft" update_rate="1000.0"/>
-    <!-- <xacro:force_torque_sensor_gazebo name="ankle_left_ft" update_rate="1000.0"/>
-    <xacro:force_torque_sensor_gazebo name="ankle_right_ft" update_rate="1000.0"/> -->
+    <xacro:force_torque_sensor_gazebo name="ankle_left_ft" update_rate="1000.0"/>
+    <xacro:force_torque_sensor_gazebo name="ankle_right_ft" update_rate="1000.0"/>
   </xacro:macro>
 </robot>

File: talos_description/urdf/sensors/ftsensor.gazebo.xacro (robot description, xacro)
@@ -15,6 +15,8 @@
   <xacro:macro name="force_torque_sensor_gazebo" params="name update_rate">
     <gazebo reference="${name}_joint">
+      <provideFeedback>true</provideFeedback>
       <preserveFixedJoint>true</preserveFixedJoint> <!-- in case this is in a fixed joint -->
       <sensor name="${name}_sensor" type="force_torque">
+        <always_on>1</always_on>
         <update_rate>${update_rate}</update_rate>
         <visualize>true</visualize>

File: talos_description/urdf/talos_full_common.urdf.xacro (robot description, xacro)
@@ -44,4 +44,6 @@
   <xacro:talos_leg prefix="left"  reflect="1" flexibility="$(arg flexibility)"/>
   <xacro:talos_leg prefix="right" reflect="-1" flexibility="$(arg flexibility)"/>
+  <xacro:ft_sensor name="ankle" parent="leg_right_6_link" side="right" reflect="1"  />
+  <xacro:ft_sensor name="ankle" parent="leg_left_6_link"  side="left"  reflect="-1" />
   <xacro:talos_addons/>
   <xacro:talos_gazebo/>

File: talos_description_inertial/urdf/inertial.xacro (robot description, xacro)
@@ -295,4 +295,18 @@
     </inertial>
   </xacro:macro>
+  <xacro:macro name="ankle_left_ft_link_inertial">
+    <inertial>
+      <mass value="0.095"/>
+      <inertia ixx="1.108502e-05" ixy="9.9077e-07" ixz="-2.3811e-07" iyy="1.092725e-05" iyz="2.3137e-07" izz="1.898772e-05" />
+      <origin rpy="0 0 0" xyz="-0.001001 0.000995 -0.008108"/>
+    </inertial>
+  </xacro:macro>
+  <xacro:macro name="ankle_left_ft_tool_link_inertial">
+    <inertial>
+      <mass value="0.001"/>
+      <inertia ixx="0" ixy="0" ixz="0" iyy="0" iyz="0" izz="0" />
+      <origin rpy="0 0 0" xyz="0 0 0"/>
+    </inertial>
+  </xacro:macro>
   <xacro:macro name="leg_right_1_link_inertial">
     <inertial>
@@ -337,4 +351,18 @@
     </inertial>
   </xacro:macro>
+  <xacro:macro name="ankle_right_ft_link_inertial">
+    <inertial>
+      <mass value="0.095"/>
+      <inertia ixx="1.108502e-05" ixy="9.9077e-07" ixz="-2.3811e-07" iyy="1.092725e-05" iyz="2.3137e-07" izz="1.898772e-05" />
+      <origin rpy="0 0 0" xyz="-0.001001 0.000995 -0.008108"/>
+    </inertial>
+  </xacro:macro>
+  <xacro:macro name="ankle_right_ft_tool_link_inertial">
+    <inertial>
+      <mass value="0.001"/>
+      <inertia ixx="0" ixy="0" ixz="0" iyy="0" iyz="0" izz="0" />
+      <origin rpy="0 0 0" xyz="0 0 0"/>
+    </inertial>
+  </xacro:macro>
   <xacro:macro name="rgbd_link_inertial">
     <inertial>

Commit message: add force sensor at the feet

File: talos_description/gazebo/gazebo.urdf.xacro (robot description, xacro)
@@ -18,6 +18,5 @@
     <gazebo>
       <plugin filename="libgazebo_ros2_control.so" name="gazebo_ros2_control">
-        <!-- in the future move this param file somewhere else -->
-        <parameters>$(find talos_controller_configuration)/config/gazebo_controller_manager_cfg.yaml</parameters>
+        <parameters>$(find talos_description)/config/gazebo_controller_manager_cfg.yaml</parameters>
         <xacro:if value="${is_multiple}">
           <!-- Do something about multirobot -->
@@ -28,9 +27,23 @@
       </plugin>
     </gazebo>
+    <gazebo>
+      <plugin name="gazebo_ros_ft" filename="libgazebo_ros_ft_sensor.so">
+        <ros>
+          <!-- Add namespace and remap the default topic -->
+          <namespace>/talos</namespace>
+          <remapping>wrench:=base_link_wrench</remapping>
+        </ros>
+        <!-- Replace camelCase elements with camel_case ones -->
+        <body_name>base_link</body_name>
+        <frame_name>link</frame_name>
+        <update_rate>1000</update_rate>
+        <gaussian_noise>0.01</gaussian_noise>
+      </plugin>
+    </gazebo>
     <xacro:imu_sensor_gazebo update_rate="1000.0"/>
-    <xacro:force_torque_sensor_gazebo name="wrist_left_ft" update_rate="1000.0"/>
-    <xacro:force_torque_sensor_gazebo name="wrist_right_ft" update_rate="1000.0"/>
-    <xacro:force_torque_sensor_gazebo name="ankle_left_ft" update_rate="1000.0"/>
-    <xacro:force_torque_sensor_gazebo name="ankle_right_ft" update_rate="1000.0"/>
+    <xacro:force_torque_sensor_gazebo parent_joint_name="wrist_left_ft_joint" sensor_name="wrist_left_ft_sensor" update_rate="1000.0"/>
+    <xacro:force_torque_sensor_gazebo parent_joint_name="wrist_right_ft_joint" sensor_name="wrist_right_ft_sensor" update_rate="1000.0"/>
+    <xacro:force_torque_sensor_gazebo parent_joint_name="leg_left_6_joint" sensor_name="ankle_left_ft_sensor" update_rate="1000.0"/>
+    <xacro:force_torque_sensor_gazebo parent_joint_name="leg_right_6_joint" sensor_name="ankle_right_ft_sensor" update_rate="1000.0"/>
   </xacro:macro>
 </robot>

File: talos_description/ros2_control/ros2_control.urdf.xacro (robot description, xacro)
@@ -66,8 +66,8 @@
       <xacro:ros2_control_torso name="torso" number="2"/>
       <!-- Force Torque sensor-->
-      <xacro:ros2_control_force_torque_sensor name="wrist_right_ft_sensor"/>
-      <xacro:ros2_control_force_torque_sensor name="wrist_left_ft_sensor"/>
-      <xacro:ros2_control_force_torque_sensor name="ankle_right_ft_sensor"/>
-      <xacro:ros2_control_force_torque_sensor name="ankle_left_ft_sensor"/>
+      <xacro:ros2_control_force_torque_sensor name="wrist" side="right"/>
+      <xacro:ros2_control_force_torque_sensor name="wrist" side="left"/>
+      <xacro:ros2_control_force_torque_sensor name="ankle" side="right"/>
+      <xacro:ros2_control_force_torque_sensor name="ankle" side="left"/>
       <!-- Leg left -->
       <xacro:ros2_control_leg side="left" number="1" />

File: talos_description/urdf/sensors/ftsensor.gazebo.xacro (robot description, xacro)
@@ -13,10 +13,10 @@
  -->
 <robot xmlns:xacro="http://ros.org/wiki/xacro">
-  <xacro:macro name="force_torque_sensor_gazebo" params="name update_rate">
-    <gazebo reference="${name}_joint">
+  <xacro:macro name="force_torque_sensor_gazebo" params="parent_joint_name sensor_name update_rate">
+    <gazebo reference="${parent_joint_name}">
       <provideFeedback>true</provideFeedback>
       <preserveFixedJoint>true</preserveFixedJoint> <!-- in case this is in a fixed joint -->
-      <sensor name="${name}_sensor" type="force_torque">
-        <always_on>1</always_on>
+      <sensor name="${sensor_name}" type="force_torque">
+        <always_on>true</always_on>
         <update_rate>${update_rate}</update_rate>
         <visualize>true</visualize>

File: talos_description/urdf/sensors/ftsensor.ros2_control.xacro (robot description, xacro)
@@ -13,6 +13,6 @@
  -->
 <robot xmlns:xacro="http://ros.org/wiki/xacro">
-  <xacro:macro name="ros2_control_force_torque_sensor" params="name">
-    <sensor name="${name}">
+  <xacro:macro name="ros2_control_force_torque_sensor" params="name side">
+    <sensor name="${name}_${side}_ft_sensor">
       <state_interface name="force.x"/>
       <state_interface name="force.y"/>

File: talos_description/urdf/talos_full_common.urdf.xacro (robot description, xacro)
@@ -44,6 +44,4 @@
   <xacro:talos_leg prefix="left"  reflect="1" flexibility="$(arg flexibility)"/>
   <xacro:talos_leg prefix="right" reflect="-1" flexibility="$(arg flexibility)"/>
-  <xacro:ft_sensor name="ankle" parent="leg_right_6_link" side="right" reflect="1"  />
-  <xacro:ft_sensor name="ankle" parent="leg_left_6_link"  side="left"  reflect="-1" />
   <xacro:talos_addons/>
   <xacro:talos_gazebo/>

File: talos_description_inertial/urdf/inertial.xacro (robot description, xacro)
@@ -297,4 +297,95 @@
   <xacro:macro name="ankle_left_ft_link_inertial">
     <inertial>
+      <mass value="0.00000001"/>
+      <inertia ixx="0" ixy="0" ixz="0" iyy="0" iyz="0" izz="0" />
+      <origin rpy="0 0 0" xyz="0 0 0"/>
+    </inertial>
+  </xacro:macro>
+  <xacro:macro name="leg_right_1_link_inertial">
+    <inertial>
+      <mass value="2.235009"/>
+      <inertia ixx="0.01049849" ixy="0.00004097" ixz="0.00009771" iyy="0.00534086" iyz="-0.0011949" izz="0.00708595" />
+      <origin rpy="0 0 0" xyz="0.08472839 -0.10997434 0.01705898"/>
+    </inertial>
+  </xacro:macro>
+  <xacro:macro name="leg_right_2_link_inertial">
+    <inertial>
+      <mass value="1.490952"/>
+      <inertia ixx="0.00497152259" ixy="0.0001311358" ixz="-4.86648e-06" iyy="0.00190550993" iyz="-4.585381e-05" izz="0.00474289754" />
+      <origin rpy="0 0 0" xyz="-0.00704703 -0.02592659 0.00273385"/>
+    </inertial>
+  </xacro:macro>
+  <xacro:macro name="leg_right_3_link_inertial">
+    <inertial>
+      <mass value="6.239871"/>
+      <inertia ixx="0.15337403915" ixy="-0.00068913396" ixz="0.00168034366" iyy="0.13648139346" iyz="0.02187635445" izz="0.03001594885" />
+      <origin rpy="0 0 0" xyz="0.0058523 -0.0636967 -0.18339564"/>
+    </inertial>
+  </xacro:macro>
+  <xacro:macro name="leg_right_4_link_inertial">
+    <inertial>
+      <mass value="3.759951"/>
+      <inertia ixx="0.04287677484" ixy="-0.00043705397" ixz="0.00078292368" iyy="0.03598906971" iyz="-0.00037717694" izz="0.01364791564" />
+      <origin rpy="0 0 0" xyz="0.01317717 -0.02917508 -0.11594602"/>
+    </inertial>
+  </xacro:macro>
+  <xacro:macro name="leg_right_5_link_inertial">
+    <inertial>
+      <mass value="1.29096"/>
+      <inertia ixx="0.01143430819" ixy="-0.00096978273" ixz="0.00039976581" iyy="0.00888974312" iyz="0.00277808667" izz="0.00506373875" />
+      <origin rpy="0 0 0" xyz="-0.01400838 -0.04180064 0.03820186"/>
+    </inertial>
+  </xacro:macro>
+  <xacro:macro name="leg_right_6_link_inertial">
+    <inertial>
+      <mass value="1.597773"/>
+      <inertia ixx="0.00439027267" ixy="6.743674e-05" ixz="0.00113816363" iyy="0.00743063029" iyz="-3.943143e-05" izz="0.00550906699" />
+      <origin rpy="0 0 0" xyz="-0.02034668 0.00051514 -0.05987428"/>
+    </inertial>
+  </xacro:macro>
+  <xacro:macro name="ankle_right_ft_link_inertial">
+    <inertial>
+      <mass value="0.00000001"/>
+      <inertia ixx="0" ixy="0" ixz="0" iyy="0" iyz="0" izz="0" />
+      <origin rpy="0 0 0" xyz="0 0 0"/>
+    </inertial>
+  </xacro:macro>
+  <xacro:macro name="rgbd_link_inertial">
+    <inertial>
+      <mass value="0.01"/>
+      <inertia ixx="3e-05" ixy="0" ixz="0" iyy="2e-06" iyz="0" izz="3e-05" />
+      <origin xyz="-0.01 0.0025 0" rpy="0 0 0"/>
+    </inertial>
+  </xacro:macro>
+  <xacro:macro name="rgbd_optical_frame_inertial">
+    <inertial>
+      <mass value="0.01"/>
+      <inertia ixx="0" ixy="0" ixz="0" iyy="0" iyz="0" izz="0" />
+      <origin rpy="0 0 0" xyz="0 0 0"/>
+    </inertial>
+  </xacro:macro>
+  <xacro:macro name="right_sole_link_inertial">
+    <inertial>
+      <mass value="0.01"/>
+      <inertia ixx="0.0001" ixy="0" ixz="0" iyy="0.0001" iyz="0" izz="0.0001" />
+      <origin rpy="0 0 0" xyz="0 0 0"/>
+    </inertial>
+  </xacro:macro>
+  <xacro:macro name="torso_1_link_inertial">
+    <inertial>
+      <mass value="2.294658"/>
+      <inertia ixx="0.00638508087" ixy="-7.107e-08" ixz="-3.065592e-05" iyy="0.00410256102" iyz="-1.46946e-06" izz="0.00622968815" />
+      <origin rpy="0 0 0" xyz="0.00078223 3.528e-05 -0.01782457"/>
+    </inertial>
+  </xacro:macro>
+  <xacro:macro name="torso_2_link_inertial">
+    <inertial>
+      <mass value="16.97403"/>
+      <inertia ixx="0.44372633826" ixy="0.00069132133" ixz="-0.01218206353" iyy="0.2998576068" iyz="-0.00019623338" izz="0.32201554742" />
+      <origin rpy="0 0 0" xyz="-0.0463563 -0.00099023 0.1452805"/>
+    </inertial>
+  </xacro:macro>
+  <xacro:macro name="wrist_left_ft_link_inertial">
+    <inertial>
       <mass value="0.095"/>
       <inertia ixx="1.108502e-05" ixy="9.9077e-07" ixz="-2.3811e-07" iyy="1.092725e-05" iyz="2.3137e-07" izz="1.898772e-05" />
@@ -302,5 +393,5 @@
     </inertial>
   </xacro:macro>
-  <xacro:macro name="ankle_left_ft_tool_link_inertial">
+  <xacro:macro name="wrist_left_ft_tool_link_inertial">
     <inertial>
       <mass value="0.001"/>
@@ -309,47 +400,5 @@
     </inertial>
   </xacro:macro>
-  <xacro:macro name="leg_right_1_link_inertial">
-    <inertial>
-      <mass value="2.235009"/>
-      <inertia ixx="0.01049849" ixy="0.00004097" ixz="0.00009771" iyy="0.00534086" iyz="-0.0011949" izz="0.00708595" />
-      <origin rpy="0 0 0" xyz="0.08472839 -0.10997434 0.01705898"/>
-    </inertial>
-  </xacro:macro>
-  <xacro:macro name="leg_right_2_link_inertial">
-    <inertial>
-      <mass value="1.490952"/>
-      <inertia ixx="0.00497152259" ixy="0.0001311358" ixz="-4.86648e-06" iyy="0.00190550993" iyz="-4.585381e-05" izz="0.00474289754" />
-      <origin rpy="0 0 0" xyz="-0.00704703 -0.02592659 0.00273385"/>
-    </inertial>
-  </xacro:macro>
-  <xacro:macro name="leg_right_3_link_inertial">
-    <inertial>
-      <mass value="6.239871"/>
-      <inertia ixx="0.15337403915" ixy="-0.00068913396" ixz="0.00168034366" iyy="0.13648139346" iyz="0.02187635445" izz="0.03001594885" />
-      <origin rpy="0 0 0" xyz="0.0058523 -0.0636967 -0.18339564"/>
-    </inertial>
-  </xacro:macro>
-  <xacro:macro name="leg_right_4_link_inertial">
-    <inertial>
-      <mass value="3.759951"/>
-      <inertia ixx="0.04287677484" ixy="-0.00043705397" ixz="0.00078292368" iyy="0.03598906971" iyz="-0.00037717694" izz="0.01364791564" />
-      <origin rpy="0 0 0" xyz="0.01317717 -0.02917508 -0.11594602"/>
-    </inertial>
-  </xacro:macro>
-  <xacro:macro name="leg_right_5_link_inertial">
-    <inertial>
-      <mass value="1.29096"/>
-      <inertia ixx="0.01143430819" ixy="-0.00096978273" ixz="0.00039976581" iyy="0.00888974312" iyz="0.00277808667" izz="0.00506373875" />
-      <origin rpy="0 0 0" xyz="-0.01400838 -0.04180064 0.03820186"/>
-    </inertial>
-  </xacro:macro>
-  <xacro:macro name="leg_right_6_link_inertial">
-    <inertial>
-      <mass value="1.597773"/>
-      <inertia ixx="0.00439027267" ixy="6.743674e-05" ixz="0.00113816363" iyy="0.00743063029" iyz="-3.943143e-05" izz="0.00550906699" />
-      <origin rpy="0 0 0" xyz="-0.02034668 0.00051514 -0.05987428"/>
-    </inertial>
-  </xacro:macro>
-  <xacro:macro name="ankle_right_ft_link_inertial">
+  <xacro:macro name="wrist_right_ft_link_inertial">
     <inertial>
       <mass value="0.095"/>
@@ -358,5 +407,5 @@
     </inertial>
   </xacro:macro>
-  <xacro:macro name="ankle_right_ft_tool_link_inertial">
+  <xacro:macro name="wrist_right_ft_tool_link_inertial">
     <inertial>
       <mass value="0.001"/>
@@ -365,66 +414,3 @@
     </inertial>
   </xacro:macro>
-  <xacro:macro name="rgbd_link_inertial">
-    <inertial>
-      <mass value="0.01"/>
-      <inertia ixx="3e-05" ixy="0" ixz="0" iyy="2e-06" iyz="0" izz="3e-05" />
-      <origin xyz="-0.01 0.0025 0" rpy="0 0 0"/>
-    </inertial>
-  </xacro:macro>
-  <xacro:macro name="rgbd_optical_frame_inertial">
-    <inertial>
-      <mass value="0.01"/>
-      <inertia ixx="0" ixy="0" ixz="0" iyy="0" iyz="0" izz="0" />
-      <origin rpy="0 0 0" xyz="0 0 0"/>
-    </inertial>
-  </xacro:macro>
-  <xacro:macro name="right_sole_link_inertial">
-    <inertial>
-      <mass value="0.01"/>
-      <inertia ixx="0.0001" ixy="0" ixz="0" iyy="0.0001" iyz="0" izz="0.0001" />
-      <origin rpy="0 0 0" xyz="0 0 0"/>
-    </inertial>
-  </xacro:macro>
-  <xacro:macro name="torso_1_link_inertial">
-    <inertial>
-      <mass value="2.294658"/>
-      <inertia ixx="0.00638508087" ixy="-7.107e-08" ixz="-3.065592e-05" iyy="0.00410256102" iyz="-1.46946e-06" izz="0.00622968815" />
-      <origin rpy="0 0 0" xyz="0.00078223 3.528e-05 -0.01782457"/>
-    </inertial>
-  </xacro:macro>
-  <xacro:macro name="torso_2_link_inertial">
-    <inertial>
-      <mass value="16.97403"/>
-      <inertia ixx="0.44372633826" ixy="0.00069132133" ixz="-0.01218206353" iyy="0.2998576068" iyz="-0.00019623338" izz="0.32201554742" />
-      <origin rpy="0 0 0" xyz="-0.0463563 -0.00099023 0.1452805"/>
-    </inertial>
-  </xacro:macro>
-  <xacro:macro name="wrist_left_ft_link_inertial">
-    <inertial>
-      <mass value="0.095"/>
-      <inertia ixx="1.108502e-05" ixy="9.9077e-07" ixz="-2.3811e-07" iyy="1.092725e-05" iyz="2.3137e-07" izz="1.898772e-05" />
-      <origin rpy="0 0 0" xyz="-0.001001 0.000995 -0.008108"/>
-    </inertial>
-  </xacro:macro>
-  <xacro:macro name="wrist_left_ft_tool_link_inertial">
-    <inertial>
-      <mass value="0.001"/>
-      <inertia ixx="0" ixy="0" ixz="0" iyy="0" iyz="0" izz="0" />
-      <origin rpy="0 0 0" xyz="0 0 0"/>
-    </inertial>
-  </xacro:macro>
-  <xacro:macro name="wrist_right_ft_link_inertial">
-    <inertial>
-      <mass value="0.095"/>
-      <inertia ixx="1.108502e-05" ixy="9.9077e-07" ixz="-2.3811e-07" iyy="1.092725e-05" iyz="2.3137e-07" izz="1.898772e-05" />
-      <origin rpy="0 0 0" xyz="-0.001001 0.000995 -0.008108"/>
-    </inertial>
-  </xacro:macro>
-  <xacro:macro name="wrist_right_ft_tool_link_inertial">
-    <inertial>
-      <mass value="0.001"/>
-      <inertia ixx="0" ixy="0" ixz="0" iyy="0" iyz="0" izz="0" />
-      <origin rpy="0 0 0" xyz="0 0 0"/>
-    </inertial>
-  </xacro:macro>
 </robot>
