Commit message: Add the possibility to start the simulation with a fixed base or not.

File: talos_description/urdf/talos_full_common.urdf.xacro (robot description, xacro)
@@ -11,4 +11,9 @@
         xmlns:controller="http://playerstage.sourceforge.net/gazebo/xmlschema/#controller"
         xmlns:interface="http://playerstage.sourceforge.net/gazebo/xmlschema/#interface">
+  <xacro:arg name="enable_crane" default="false"/>
+  <xacro:arg name="use_fixed_base" default="false"/>
+  <xacro:arg name="use_sim" default="false"/>
+  <xacro:arg name="multiple" default="false"/>
+  <xacro:property name="is_multiple" value="$(arg multiple)" />
   <xacro:if value="$(arg enable_crane)">
     <xacro:include filename="$(find talos_description)/urdf/crane/crane.urdf.xacro" />
@@ -28,11 +33,17 @@
   <!-- Materials for visualization -->
   <xacro:include filename="$(find talos_description)/urdf/materials.urdf.xacro" />
+  <!-- Fixed world frame -->
+  <xacro:if value="$(arg use_fixed_base)">
+    <link name="world"/>
+    <joint name="world_fixed" type="fixed">
+        <origin xyz="0 0 0" rpy="0 0 0"/>
+        <parent link="world"/>
+        <child link="base_link"/>
+    </joint>
+  </xacro:if>
   <xacro:talos_torso name="torso" />
   <xacro:if value="$(arg enable_crane)">
     <xacro:crane parent="torso_2_link"/>
   </xacro:if>
-  <xacro:arg name="use_sim" default="false"/>
-  <xacro:arg name="multiple" default="false"/>
-  <xacro:property name="is_multiple" value="$(arg multiple)" />
   <xacro:talos_head name="head" parent="torso_2_link" disable_gazebo_camera="$(arg disable_gazebo_camera)" head_type="$(arg head_type)"/>
   <xacro:talos_arm name="arm" parent="torso_2_link" side="left" reflect="1" />

File: talos_description/urdf/torso/torso.urdf.xacro (robot description, xacro)
@@ -17,11 +17,4 @@
     <xacro:include filename="$(find talos_description)/test/calibration/calibration_constants.urdf.xacro" />
   </xacro:if>
-  <!-- Fixed world frame -->
-  <link name="world"/>
-  <joint name="world_fixed" type="fixed">
-      <origin xyz="0 0 0" rpy="0 0 0"/>
-      <parent link="world"/>
-      <child link="base_link"/>
-  </joint>
  <!--Constant parameters-->
   <xacro:property name="torso_max_vel"  value="5.4" />
