Commit message: fix torso and head ros2_control

File: talos_description/ros2_control/ros2_control.urdf.xacro (robot description, xacro)
@@ -61,4 +61,6 @@
       <!-- Head -->
       <xacro:ros2_control_head name="head" offset_value_1="${head_1_joint_yaw_offset}" offset_value_2="${head_2_joint_yaw_offset}"/>
+      <!-- Torso -->
+      <xacro:ros2_control_torso name="torso"/>
        <!-- Force Torque sensor-->
       <xacro:ros2_control_force_torque_sensor name="wrist_right_ft_sensor"/>

File: talos_description/urdf/head/head.ros2_control.xacro (robot description, xacro)
@@ -14,5 +14,13 @@
 <robot xmlns:xacro="http://ros.org/wiki/xacro">
   <xacro:macro name="ros2_control_head" params="name offset_value_1 offset_value_2" >
-    <joint name="${name}_joint">
+    <joint name="${name}_1_joint">
+      <command_interface name="position" />
+      <command_interface name="velocity" />
+      <command_interface name="effort" />
+      <state_interface name="position" />
+      <state_interface name="velocity" />
+      <state_interface name="effort" />
+    </joint>
+    <joint name="${name}_2_joint">
       <command_interface name="position" />
       <command_interface name="velocity" />

File: talos_description/urdf/torso/torso.ros2_control.xacro (robot description, xacro)
@@ -14,5 +14,13 @@
 <robot xmlns:xacro="http://ros.org/wiki/xacro">
   <xacro:macro name="ros2_control_torso" params="name" >
-    <joint name="${name}_joint">
+    <joint name="${name}_1_joint">
+      <command_interface name="position" />
+      <command_interface name="velocity" />
+      <command_interface name="effort" />
+      <state_interface name="position" />
+      <state_interface name="velocity" />
+      <state_interface name="effort" />
+    </joint>
+    <joint name="${name}_2_joint">
       <command_interface name="position" />
       <command_interface name="velocity" />

Commit message: fix the arm transmission ros2_control xacro

File: talos_description/ros2_control/ros2_control.urdf.xacro (robot description, xacro)
@@ -23,4 +23,5 @@
     <xacro:include filename="$(find talos_description)/urdf/sensors/imu.ros2_control.xacro" />
     <xacro:include filename="$(find talos_description)/urdf/sensors/ftsensor.ros2_control.xacro" />
+    <xacro:include filename="$(find talos_description_calibration)/urdf/calibration/calibration_constants.urdf.xacro" />
     <!-- Calibration offsets -->
     <xacro:include filename="$(find talos_description_calibration)/urdf/calibration/calibration_constants.urdf.xacro" />
@@ -39,8 +40,8 @@
       </xacro:if>
       <!-- arm right-->
-      <xacro:ros2_control_arm name="arm" side="right" number="1"/>
-      <xacro:ros2_control_arm name="arm" side="right" number="2"/>
-      <xacro:ros2_control_arm name="arm" side="right" number="3"/>
-      <xacro:ros2_control_arm name="arm" side="right" number="4"/>
+      <xacro:ros2_control_arm name="arm" side="right" number="1" joint_offset="${arm_right_1_joint_offset}"/>
+      <xacro:ros2_control_arm name="arm" side="right" number="2" joint_offset="${arm_right_2_joint_offset}"/>
+      <xacro:ros2_control_arm name="arm" side="right" number="3" joint_offset="${arm_right_3_joint_offset}"/>
+      <xacro:ros2_control_arm name="arm" side="right" number="4" joint_offset="${arm_right_4_joint_offset}"/>
       <!-- Wrist right -->
       <xacro:ros2_control_wrist name="arm" side="right" number="5"/>
@@ -48,8 +49,8 @@
       <xacro:ros2_control_wrist name="arm" side="right" number="7"/>
       <!-- Arm left-->
-      <xacro:ros2_control_arm name="arm" side="left" number="1"/>
-      <xacro:ros2_control_arm name="arm" side="left" number="2"/>
-      <xacro:ros2_control_arm name="arm" side="left" number="3"/>
-      <xacro:ros2_control_arm name="arm" side="left" number="4"/>
+      <xacro:ros2_control_arm name="arm" side="left" number="1" joint_offset="${arm_left_1_joint_offset}"/>
+      <xacro:ros2_control_arm name="arm" side="left" number="2" joint_offset="${arm_left_2_joint_offset}"/>
+      <xacro:ros2_control_arm name="arm" side="left" number="3" joint_offset="${arm_left_3_joint_offset}"/>
+      <xacro:ros2_control_arm name="arm" side="left" number="4" joint_offset="${arm_left_4_joint_offset}"/>
       <!-- Wrist left -->
       <xacro:ros2_control_wrist name="arm" side="left" number="5"/>

File: talos_description/urdf/arm/arm.ros2_control.xacro (robot description, xacro)
@@ -13,5 +13,7 @@
  -->
 <robot xmlns:xacro="http://ros.org/wiki/xacro">
-  <xacro:macro name="ros2_control_arm" params="name side number" >
+  <!--File includes-->
+  <xacro:include filename="$(find talos_description)/urdf/arm/arm.transmission.xacro" />
+  <xacro:macro name="ros2_control_arm" params="name side number joint_offset" >
     <joint name="${name}_${side}_${number}_joint">
       <command_interface name="position" />
@@ -23,5 +25,5 @@
     </joint>
    <!-- transmissions -->
-  <xacro:include filename="$(find talos_description)/urdf/arm/${side}_arm.transmissions.urdf.xacro" />
+  <xacro:talos_arm_simple_transmission name="${name}" side="${side}" number="${number}" reduction="1.0" offset_value="${joint_offset}"/>
   </xacro:macro>
 </robot>

Commit message: Fix the wrist transmission of the ros2_control xacro

File: talos_description/ros2_control/ros2_control.urdf.xacro (robot description, xacro)
@@ -45,7 +45,5 @@
       <xacro:ros2_control_arm name="arm" side="right" number="4" joint_offset="${arm_right_4_joint_offset}"/>
       <!-- Wrist right -->
-      <xacro:ros2_control_wrist name="arm" side="right" number="5"/>
-      <xacro:ros2_control_wrist name="arm" side="right" number="6"/>
-      <xacro:ros2_control_wrist name="arm" side="right" number="7"/>
+      <xacro:ros2_control_wrist name="arm" side="right" joint_5_offset="${arm_right_5_joint_offset}" joint_6_offset="${arm_right_6_joint_offset}" joint_7_offset="${arm_right_7_joint_offset}"/>
       <!-- Arm left-->
       <xacro:ros2_control_arm name="arm" side="left" number="1" joint_offset="${arm_left_1_joint_offset}"/>
@@ -54,7 +52,5 @@
       <xacro:ros2_control_arm name="arm" side="left" number="4" joint_offset="${arm_left_4_joint_offset}"/>
       <!-- Wrist left -->
-      <xacro:ros2_control_wrist name="arm" side="left" number="5"/>
-      <xacro:ros2_control_wrist name="arm" side="left" number="6"/>
-      <xacro:ros2_control_wrist name="arm" side="left" number="7"/>
+      <xacro:ros2_control_wrist name="arm" side="left" joint_5_offset="${arm_left_5_joint_offset}" joint_6_offset="${arm_left_6_joint_offset}" joint_7_offset="${arm_left_7_joint_offset}"/>
       <!-- Gripper right-->
       <xacro:ros2_control_gripper name="gripper_right"/>

File: talos_description/urdf/arm/wrist.ros2_control.xacro (robot description, xacro)
@@ -13,6 +13,8 @@
  -->
 <robot xmlns:xacro="http://ros.org/wiki/xacro">
-  <xacro:macro name="ros2_control_wrist" params="name side number" >
-    <joint name="${name}_${side}_${number}_joint">
+  <!--File includes-->
+  <xacro:include filename="$(find talos_description)/urdf/arm/wrist.transmission.xacro" />
+  <xacro:macro name="ros2_control_wrist" params="name side joint_5_offset joint_6_offset joint_7_offset" >
+    <joint name="${name}_${side}_5_joint">
       <command_interface name="position" />
       <command_interface name="velocity" />
@@ -22,6 +24,28 @@
       <state_interface name="effort" />
     </joint>
-   <!-- transmissions -->
-   <xacro:include filename="$(find talos_description)/urdf/arm/${side}_wrist.transmissions.urdf.xacro" />
+    <joint name="${name}_${side}_6_joint">
+      <command_interface name="position" />
+      <command_interface name="velocity" />
+      <command_interface name="effort" />
+      <state_interface name="position" />
+      <state_interface name="velocity" />
+      <state_interface name="effort" />
+    </joint>
+    <joint name="${name}_${side}_7_joint">
+      <command_interface name="position" />
+      <command_interface name="velocity" />
+      <command_interface name="effort" />
+      <state_interface name="position" />
+      <state_interface name="velocity" />
+      <state_interface name="effort" />
+    </joint>
+    <!-- transmissions -->
+  <xacro:talos_wrist_simple_transmission name="${name}" side="${side}" number="5" reduction="1.0"
+                                         offset_value="${joint_5_offset}"/>
+  <xacro:talos_wrist_differential_transmission name="${name}" side="${side}" number_1="6" number_2="7"
+                                                act_reduction_1="-1.0" act_reduction_2="1.0"
+                                                jnt_reduction_1="-1.0" jnt_reduction_2="-1.0"
+                                                offset_value_1="${joint_6_offset}"
+                                                offset_value_2="${joint_7_offset}"/>
   </xacro:macro>
 </robot>

Commit message: Fix the torso transmission duplication in ros2_control xacro

File: talos_description/ros2_control/ros2_control.urdf.xacro (robot description, xacro)
@@ -60,6 +60,5 @@
       <xacro:ros2_control_head name="head" number_1="1" number_2="2" offset_value_1="${head_1_joint_yaw_offset}" offset_value_2="${head_2_joint_yaw_offset}"/>
       <!-- Torso -->
-      <xacro:ros2_control_torso name="torso" number="1"/>
-      <xacro:ros2_control_torso name="torso" number="2"/>
+      <xacro:ros2_control_torso name="torso"/>
       <!-- Force Torque sensor-->
       <xacro:ros2_control_force_torque_sensor name="wrist" side="right"/>

File: talos_description/urdf/torso/torso.ros2_control.xacro (robot description, xacro)
@@ -13,6 +13,14 @@
  -->
 <robot xmlns:xacro="http://ros.org/wiki/xacro">
-  <xacro:macro name="ros2_control_torso" params="name number" >
-    <joint name="${name}_${number}_joint">
+  <xacro:macro name="ros2_control_torso" params="name joint_1:='1' joint_2:='2'">
+    <joint name="${name}_${joint_1}_joint">
+      <command_interface name="position" />
+      <command_interface name="velocity" />
+      <command_interface name="effort" />
+      <state_interface name="position" />
+      <state_interface name="velocity" />
+      <state_interface name="effort" />
+    </joint>
+    <joint name="${name}_${joint_2}_joint">
       <command_interface name="position" />
       <command_interface name="velocity" />
@@ -24,5 +32,5 @@
     <!-- transmissions -->
     <xacro:include filename="$(find talos_description)/urdf/torso/torso.transmission.xacro" />
-    <xacro:talos_torso_differential_transmission name="${name}" number1="1" number2="2"
+    <xacro:talos_torso_differential_transmission name="${name}" number1="${joint_1}" number2="${joint_2}"
                                                 act_reduction1="1.0" act_reduction2="1.0"
                                                 jnt_reduction1="1.0" jnt_reduction2="1.0" />
