Commit message: Commenting gripper mimic joints not working in real robot

File: talos_description/urdf/gripper/gripper.ros2_control.xacro (robot description, xacro)
@@ -14,5 +14,5 @@
 <robot xmlns:xacro="http://ros.org/wiki/xacro">
   <xacro:macro name="ros2_control_gripper" params="name" >
-    <xacro:macro name="ros2_control_talos_gripper_mimic_joint" params="mimic_joint_name actuated_joint_name multiplier" >
+    <!-- <xacro:macro name="ros2_control_talos_gripper_mimic_joint" params="mimic_joint_name actuated_joint_name multiplier" >
       <joint name="${mimic_joint_name}">
         <param name="mimic">${actuated_joint_name}</param>
@@ -25,5 +25,5 @@
         <state_interface name="effort" />
       </joint>
-    </xacro:macro>
+    </xacro:macro> -->
     <joint name="${name}_joint">
       <command_interface name="position" />
@@ -34,5 +34,5 @@
       <state_interface name="effort" />
     </joint>
-    <xacro:ros2_control_talos_gripper_mimic_joint mimic_joint_name="${name}_inner_double_joint"
+    <!-- <xacro:ros2_control_talos_gripper_mimic_joint mimic_joint_name="${name}_inner_double_joint"
                                                     actuated_joint_name="${name}_joint"
                                                     multiplier="1"/>
@@ -51,5 +51,5 @@
     <xacro:ros2_control_talos_gripper_mimic_joint mimic_joint_name="${name}_fingertip_3_joint"
                                                     actuated_joint_name="${name}_joint"
-                                                    multiplier="-1"/>
+                                                    multiplier="-1"/> -->
    <!-- transmissions -->
   <xacro:include filename="$(find talos_description)/urdf/gripper/gripper.transmission.xacro" />
